Commit message: urdf change

File: robot_arm/urdf/02-diff_drive.urdf (robot description, URDF)
Before this commit: robot Robot_Arm, 11 links, 10 joints
Links:
- removed link base_foot
Joints:
- removed joint base
- joint hokuyo_joint: origin xyz=0 -0.09 0 rpy=0 0 0 -> xyz=0.07 0 0.08 rpy=0 0 0
- joint left_back_wheel_joint: axis 1 0 0 -> 0 1 0; origin xyz=-0.115 -0.062 0.015 rpy=0 0 0 -> xyz=-0.058 0.115  0.015 rpy=0 0 0
- joint left_front_wheel_joint: axis 1 0 0 -> 0 1 0; origin xyz=-0.115 0.058 0.015 rpy=0 0 0 -> xyz=0.062 0.115  0.015 rpy=0 0 0
- joint right_back_wheel_joint: axis 1 0 0 -> 0 1 0; origin xyz=0.115 -0.062 0.015 rpy=0 0 0 -> xyz=-0.058 -0.115  0.015 rpy=0 0 0
- joint right_front_wheel_joint: axis 1 0 0 -> 0 1 0; origin xyz=0.115 0.058 0.015 rpy=0 0 0 -> xyz=0.062 -0.115  0.015 rpy=0 0 0

File: robot_arm/urdf/03-robot_arm.urdf (robot description, URDF)
Before this commit: robot Robot_Arm, 26 links, 25 joints
Links:
- removed link base_foot
- link elbow_pan_link: mass 0.1 -> 0.05
- link elbow_pitch_link: mass 0.1 -> 0.05
- link gripper_pan_link: mass 0.04 -> 0.01
- link gripper_pitch_link: mass 0.04 -> 0.01
- link servo_elbow_pan: mass 0.2 -> 0.05
- link servo_gripper_pan: mass 0.2 -> 0.05
- link servo_shoulder_roll: mass 0.25 -> 0.05
- link servo_wrist_roll: mass 0.2 -> 0.05
- link shoulder_pan_link: mass 0.1 -> 0.05
- link shoulder_roll_link: mass 0.1 -> 0.05
Joints:
- removed joint base
- joint elbow_pitch_joint: origin xyz=0 0 0.058 rpy=0 0 0 -> xyz=0 0 0.078 rpy=0 0 0
- joint gripper_pan_joint: origin xyz=0 0 0.1 rpy=0 0 0 -> xyz=0 0 0.09 rpy=0 0 0
- joint hokuyo_joint: origin xyz=0 -0.09 0 rpy=0 0 0 -> xyz=0.07 0 0.08 rpy=0 0 0
- joint left_back_wheel_joint: axis 1 0 0 -> 0 1 0; origin xyz=-0.115 -0.062 0.015 rpy=0 0 0 -> xyz=-0.058 0.115  0.015 rpy=0 0 0
- joint left_front_wheel_joint: axis 1 0 0 -> 0 1 0; origin xyz=-0.115 0.058 0.015 rpy=0 0 0 -> xyz=0.062 0.115  0.015 rpy=0 0 0
- joint left_gripper_joint: limit lower=0.15 upper=0.548 effort=1000.0 velocity=0.5 -> lower=0.15 upper=0.548 effort=100.0 velocity=1
- joint right_back_wheel_joint: axis 1 0 0 -> 0 1 0; origin xyz=0.115 -0.062 0.015 rpy=0 0 0 -> xyz=-0.058 -0.115  0.015 rpy=0 0 0
- joint right_front_wheel_joint: axis 1 0 0 -> 0 1 0; origin xyz=0.115 0.058 0.015 rpy=0 0 0 -> xyz=0.062 -0.115  0.015 rpy=0 0 0
- joint right_gripper_joint: limit lower=0.15 upper=0.548 effort=1000.0 velocity=0.5 -> lower=0.15 upper=0.548 effort=100.0 velocity=1
- joint servo_joint3: origin xyz=-0.004 0 0.09 rpy=0 0 0 -> xyz=-0.004 0 0.098 rpy=0 0 0
- joint servo_joint4: origin xyz=0 0 0.05 rpy=0 0 0 -> xyz=0 0 0.03 rpy=0 0 0
- joint shoulder_pan_joint: origin xyz=0 0 0.07 rpy=0 0 0 -> xyz=0 0 0.07 rpy=0 0 1.57
- joint shoulder_roll_joint: origin xyz=0 0 0.055 rpy=0 0 0 -> xyz=0 0 0.06 rpy=0 0 0
