Commit message: arm

File: robot_arm/urdf/04-robot_arm_servo.urdf.xacro (robot description, xacro)
@@ -420,5 +420,5 @@
       <joint name="${prefix}_gripper_joint" type="revolute">
       <axis xyz="${-reflect} 0 0"/>
-      <limit effort="100.0" lower="0.15" upper="0.548" velocity="1"/>
+      <limit effort="100.0" lower="0.15" upper="0.75" velocity="1"/>
       <origin rpy="0 -1.57 0" xyz="0 ${reflect*0.01} 0"/>
       <parent link="gripper_pitch_link"/>
@@ -426,6 +426,6 @@
       <safety_controller k_position="20"
                          k_velocity="20"
-                         soft_lower_limit="${-0.15 }"
-                         soft_upper_limit="${ 0.0 }"/>
+                         soft_lower_limit="${0.0 }"
+                         soft_upper_limit="${ 0.45 }"/>
     <dynamics damping="50" friction="1"/>
     </joint>
